File: 5 Lora-nodes Espressif Systems esp32/1 p1_smart_meter_TTN_Apeldoorn/esp32-p1-node-master/hardware/esp32-p1-node-board/esp32-p1-node-board/esp32-p1-node-board.sch (KiCad schematic (older format))
At the start: 18 parts, among them J1 RJ11-6, Q1 BC847, Q2 BSS138, U1 TTGO_LoRa32_V11

Commit message: Added IMN003
Parts:
- COAX1: symbol esp32_node:SMA-ANT-CONN -> esp32-p1-node-board-rescue:SMA-ANT-CONN-esp32_node
- Conn1: symbol esp32_node:THT_USB-B-Mini -> esp32-p1-node-board-rescue:THT_USB-B-Mini-esp32_node
- J1: symbol SparkFun-Connectors:RJ11-6 -> esp32-p1-node-board-rescue:RJ11-6-SparkFun-Connectors
- JP1, JP2, JP3: symbol SparkFun-Jumpers:JUMPER-SMT_3_1-NC -> esp32-p1-node-board-rescue:JUMPER-SMT_3_1-NC-SparkFun-Jumpers
- U1: symbol esp32_node:TTGO_LoRa32_V11 -> esp32-p1-node-board-rescue:TTGO_LoRa32_V11-esp32_node
Changed lines of the file:
@@
 $EndDescr
 $Comp
-L SparkFun-Connectors:RJ11-6 J1
+L esp32-p1-node-board-rescue:RJ11-6-SparkFun-Connectors J1
 U 1 1 5F00D179
 P 1200 1550
@@
 5V
 $Comp
-L esp32_node:TTGO_LoRa32_V11 U1
+L esp32-p1-node-board-rescue:TTGO_LoRa32_V11-esp32_node U1
 U 1 1 5F01626F
 P 5500 2650
@@
 TXD
 $Comp
-L SparkFun-Jumpers:JUMPER-SMT_3_1-NC JP1
+L esp32-p1-node-board-rescue:JUMPER-SMT_3_1-NC-SparkFun-Jumpers JP1
 U 1 1 5F1DD89F
 P 3550 4450
@@
 SOFT_RXD
 $Comp
-L SparkFun-Jumpers:JUMPER-SMT_3_1-NC JP2
+L esp32-p1-node-board-rescue:JUMPER-SMT_3_1-NC-SparkFun-Jumpers JP2
 U 1 1 5F1EB1BA
 P 3550 5400
@@
 	5900 5050 6600 5050
 $Comp
-L esp32_node:THT_USB-B-Mini Conn1
+L esp32-p1-node-board-rescue:THT_USB-B-Mini-esp32_node Conn1
 U 1 1 5F1FC4B8
 P 5300 5300
@@
 GND
 $Comp
-L esp32_node:SMA-ANT-CONN COAX1
+L esp32-p1-node-board-rescue:SMA-ANT-CONN-esp32_node COAX1
 U 1 1 5F1FA2D2
 P 5400 4450
@@
 $EndComp
 $Comp
-L SparkFun-Jumpers:JUMPER-SMT_3_1-NC JP3
+L esp32-p1-node-board-rescue:JUMPER-SMT_3_1-NC-SparkFun-Jumpers JP3
 U 1 1 5F231B69
 P 3550 6350
